File: epaper.kicad_sch (KiCad schematic)
At the start: 21 parts, among them J1 Conn_01x24, Q1 Si1308EDL

Commit message: hop
Other:
- note added: "100uH / 1amp"
Changed lines of the file:
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@@
+		)
+	)
+	(text "100uH / 1amp"
+		(exclude_from_sim no)
+		(at 48.514 44.704 0)
+		(effects
+			(font
+				(size 1.27 1.27)
+			)
 		)
 	)
