File: linky_panel.kicad_pcb (KiCad board)
At the start: 4 copper layers, 66 x 40 mm, 91 parts, among them J1 Conn_01x24, J2 Conn_02x05_Counter_Clockwise, J3 USB_B_Micro, J4 Conn_01x02_Pin, Q1 Si1308EDL, SW1 SW1, SW2 SW2, U1 TPS78230DDC, U2 MCP73811T-420I-OT, U3 STM32WB55RGVx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

Commit message: hop
Parts:
- removed C31, C32: 1uF, Capacitor_SMD:C_0603_1608Metric
- removed the H2 at (56.0, -6.00)
- removed kibuzzard-670FAFC9: G***, kibuzzard-670FAFC9
- removed kibuzzard-670FAFD1: G***, kibuzzard-670FAFD1
- added C33: 4.7uF, Capacitor_SMD:C_0603_1608Metric, F.Cu at (92.5, 53.2)
- added R17: 220k, Resistor_SMD:R_0402_1005Metric, F.Cu at (95.7, 54.9)
- added R18: 470k, Resistor_SMD:R_0402_1005Metric, F.Cu at (95.7, 56.9)
- added kibuzzard-6710CDD1: G***, kibuzzard-6710CDD1, F.Cu at (109.8, 63.5)
- added kibuzzard-6710CDDC: G***, kibuzzard-6710CDDC, F.Cu at (109.8, 65.6)
- TP1, TP8: moved to B.Cu
- moved H2 83.0 mm to (57.9, 64.0), turned to 180 degrees
- moved H1 67.2 mm to (73.8, 40.7), turned to 180 degrees
- moved SW2 65.4 mm to (58.9, 70.2), turned to 0 degrees
- moved SW1 65.2 mm to (112.9, 70.2), turned to 0 degrees
- moved J1 55.2 mm to (113.5, 53.2), turned to 90 degrees
- moved J2 53.6 mm to (56.9, 56.6), turned to -90 degrees
- moved JP1 51.6 mm to (111.5, 55.1), turned to 180 degrees
- moved R4 50.0 mm to (60.9, 50.8), turned to -90 degrees
- moved C28 49.6 mm to (110.0, 57.9), turned to 180 degrees
- moved C19 49.5 mm to (110.0, 45.9), turned to 0 degrees
- moved C25 49.2 mm to (110.0, 56.9), turned to 180 degrees
- moved Y2 49.1 mm to (61.8, 47.1), turned to 180 degrees
- moved C20 49.1 mm to (110.0, 47.0), turned to 0 degrees
- moved C21 48.7 mm to (110.0, 48.1), turned to 0 degrees
- moved C22 48.4 mm to (110.0, 49.2), turned to 0 degrees
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Connections:
- U3 pad 21: /wb55/pa6 -> /vbat_div
Routing:
- net /vbat_div: track 0.00 -> 32.9 mm, vias 0 -> 2
- net +BATT: track 41.2 -> 17.6 mm, vias 2 -> 8
- net +3.3V: track 13.3 -> 6.73 mm, vias 7 -> 0
- net GND: track 64.6 -> 59.4 mm, vias 100 -> 143
- net /wb55/uart_txd: track 17.1 -> 21.5 mm
- net /wb55/swclk: track 15.8 -> 11.9 mm
- net /wb55/rst: track 30.1 -> 26.6 mm
- net /wb55/swdio: track 14.1 -> 10.6 mm
- net /wb55/uart_rxd: track 18.9 -> 22.3 mm
- net /wb55/swo: track 19.8 -> 16.9 mm
- net /wb55/ant_path: track 4.41 -> 2.09 mm
- net VBUS: track 10.9 -> 13.2 mm
- net /epd_rst: track 53.9 -> 55.2 mm
- net VDD: track 37.0 -> 36.0 mm, vias 18 -> 21
- net /epaper/vdd_lcd: track 11.5 -> 10.7 mm
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- added copper zone on In2.Cu, net +BATT
- removed copper zone on In2.Cu, net +3.3V
Other:
- outline, holes or cut-outs redrawn
