File: linky_panel.kicad_sch (KiCad schematic)
At the start: 34 parts, among them J3 USB_B_Micro, J4 Conn_01x02_Pin, SW1 SW1, SW2 SW2, U1 TPS78230DDC, U2 MCP73811T-420I-OT

Commit message: hop
Parts:
- removed C31, C32: 1uF, Capacitor_SMD:C_0603_1608Metric, symbol Device:C
- added C33: 4.7uF, Capacitor_SMD:C_0603_1608Metric, symbol pspice:CAP
- added R17: 220k, Resistor_SMD:R_0402_1005Metric, symbol Device:R
- added R18: 470k, Resistor_SMD:R_0402_1005Metric, symbol Device:R
Connections:
- net +BATT: now also R17.2
- net GND: now also C33.2, R18.1
- net VBUS: now also C33.1
- new net vbat_div: R17.1, R18.2
- no-connect marks 33 -> 35
Other:
- note removed: "mesure tension d'alim ?"
- moved on the sheet: C1, C2, C3, J3, J4, JP2, R15, R16, U1, U2
